File: Keyboard_PCB.kicad_pcb (KiCad board)
At the start: 2 copper layers, 50 x 50 mm, 24 parts, among them CON1 PS/2_JACK, CON2 USB_JACK, IC1 FT232RL, U1 ATMEGA328, X1 CRYSTAL

Commit message: Added description and exported files.
Other:
- board text added: "PS/2 Keyboard rev1"
Changed lines of the file:
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@@
     (links 80)
     (no_connects 0)
-    (area 86.275 71.275 185.058333 185.725001)
+    (area 88.174999 67.150001 185.158333 185.825001)
     (thickness 1.6)
-    (drawings 6)
+    (drawings 7)
     (tracks 284)
     (zones 0)
@@
     (pad_to_mask_clearance 0)
     (aux_axis_origin 0 0)
-    (visible_elements 7FFFFDAF)
+    (visible_elements 7FFFFFBF)
     (pcbplotparams
-      (layerselection 3178497)
+      (layerselection 284196865)
       (usegerberextensions true)
-      (excludeedgelayer true)
+      (excludeedgelayer false)
       (linewidth 0.150000)
       (plotframeref false)
@@
       (outputformat 1)
       (mirror false)
-      (drillshape 1)
+      (drillshape 0)
       (scaleselection 1)
-      (outputdirectory ""))
+      (outputdirectory OUTPUT/))
   )
   (net 0 "")
@@
     )
   )
+  (gr_text "PS/2 Keyboard\nrev1" (at 120 95) (layer F.SilkS)
+    (effects (font (size 2 2) (thickness 0.25)))
+  )
   (dimension 50 (width 0.3) (layer B.SilkS)
